Commit message: collect

File: gello_teleop/models/xarm7_dynamics.urdf (robot description, URDF)
Before this commit: robot xarm7, 9 links, 8 joints
Links:
- link link1: mass 0.42603 -> 2.382
- link link2: mass 0.56095 -> 1.869
- link link3: mass 0.44463 -> 1.6383
- link link4: mass 0.52387 -> 1.7269
- link link5: mass 0.18554 -> 1.3203
- link link6: mass 0.31344 -> 1.325
- link link7: mass 0.31468 -> 0.17
